File: PCB/P2/Leviosa/Leviosa.kicad_sch (KiCad schematic)
At the start: 54 parts, among them J1 Barrel_Jack, J2 2.54mm 1x03 Spare

Commit message: add test images (various)
Parts:
- added R14, R16: 3.9kΩ, Resistor_SMD:R_0603_1608Metric, symbol Device:R_US
- Coil1: value 3.7mH -> 7.4mH
- R13, R8: value 1kΩ -> 330Ω
- V_reg1: value AMS1117-5.0 -> LM7805
Connections:
- net 5V: now also R14.2, R16.2
- net no_magnet_point_trigger: now also R16.1
- net set_point_trigger: now also R14.1
Changed lines of the file:
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@@
 	)
 	(junction
+		(at 190.5 85.09)
+		(diameter 0)
+		(color 0 0 0 0)
+	)
+	(junction
 		(at 30.48 173.99)
 		(diameter 0)
@@
 	)
 	(junction
+		(at 190.5 134.62)
+		(diameter 0)
+		(color 0 0 0 0)
+	)
+	(junction
 		(at 91.44 38.1)
 		(diameter 0)
@@
 		)
 	)
+	(label "5V"
+		(at 182.88 134.62 180)
+		(effects
+			(font
+				(size 1.27 1.27)
+			)
+			(justify right bottom)
+		)
+	)
 	(label "set_point_trigger"
 		(at 191.77 85.09 0)
@@
 		)
 	)
+	(label "5V"
+		(at 182.88 85.09 180)
+		(effects
+			(font
+				(size 1.27 1.27)
+			)
+			(justify right bottom)
+		)
+	)
 	(label "V_out"
 		(at 245.11 38.1 0)
@@
 	)
 	(symbol
+		(lib_id "Device:R_US")
+		(at 186.69 134.62 270)
+		(unit 1)
+		(exclude_from_sim no)
+		(in_bom yes)
+		(on_board yes)
+		(dnp no)
+		(property "Reference" "R16"
+			(at 186.436 130.048 90)
+			(effects
+				(font
+					(size 1.27 1.27)
+				)
+			)
+		)
+		(property "Value" "3.9kΩ"
+			(at 186.69 132.08 90)
+			(effects
+				(font
+					(size 1.27 1.27)
+				)
+			)
+		)
+		(property "Footprint" "Resistor_SMD:R_0603_1608Metric"
+			(at 186.436 135.636 90)
+			(effects
+				(font
+					(size 1.27 1.27)
+				)
+				(hide yes)
+			)
+		)
+		(property "Datasheet" "~"
+			(at 186.69 134.62 0)
+			(effects
+				(font
+					(size 1.27 1.27)
+				)
+				(hide yes)
+			)
+		)
+		(property "Description" ""
+			(at 186.69 134.62 0)
+			(effects
+				(font
+					(size 1.27 1.27)
+				)
+			)
+		)
+		(property "Link" "https://jlcpcb.com/partdetail/23745-0603WAF3901T5E/C23018"
+			(at 186.69 134.62 90)
+			(effects
+				(font
+					(size 1.27 1.27)
+				)
+				(hide yes)
+			)
+		)
+		(pin "1"
+		)
+		(pin "2"
+		)
+		(instances
+			(project "Leviosa"
+				(path "/fe766911-203b-467c-b704-d4bd488f6c98"
+					(reference "R16")
+					(unit 1)
+				)
+			)
+		)
+	)
+	(symbol
 		(lib_id "Device:C")
 		(at 234.95 67.31 0)
@@
 			)
 		)
-		(property "Value" "1kΩ"
+		(property "Value" "330Ω"
 			(at 214.63 82.55 90)
 			(effects
@@
 			)
 		)
-		(property "Value" "3.7mH"
+		(property "Value" "7.4mH"
 			(at 246.38 68.58 0)
 			(effects
@@
 			)
 		)
-		(property "Value" "AMS1117-5.0"
+		(property "Value" "LM7805"
 			(at 83.82 34.29 0)
 			(effects
@@
 			)
 		)
-		(property "Value" "1kΩ"
+		(property "Value" "330Ω"
 			(at 231.14 132.08 90)
 			(effects
@@
 					(unit 1)
 				)
+			)
+		)
+	)
+	(symbol
+		(lib_id "Device:R_US")
+		(at 186.69 85.09 270)
+		(unit 1)
+		(exclude_from_sim no)
+		(in_bom yes)
+		(on_board yes)
+		(dnp no)
+		(property "Reference" "R14"
+			(at 186.436 80.518 90)
+			(effects
+				(font
+					(size 1.27 1.27)
+				)
+			)
+		)
+		(property "Value" "3.9kΩ"
+			(at 186.69 82.55 90)
+			(effects
+				(font
+					(size 1.27 1.27)
+				)
+			)
+		)
+		(property "Footprint" "Resistor_SMD:R_0603_1608Metric"
+			(at 186.436 86.106 90)
+			(effects
+				(font
+					(size 1.27 1.27)
+				)
+				(hide yes)
+			)
+		)
+		(property "Datasheet" "~"
+			(at 186.69 85.09 0)
+			(effects
+				(font
+					(size 1.27 1.27)
+				)
+				(hide yes)
+			)
+		)
+		(property "Description" ""
+			(at 186.69 85.09 0)
+			(effects
+				(font
+					(size 1.27 1.27)
+				)
+			)
+		)
+		(property "Link" "https://jlcpcb.com/partdetail/23745-0603WAF3901T5E/C23018"
+			(at 186.69 85.09 90)
+			(effects
+				(font
+					(size 1.27 1.27)
+				)
+				(hide yes)
+			)
+		)
+		(pin "1"
+		)
+		(pin "2"
+		)
+		(instances
+			(project "Leviosa"
+				(path "/fe766911-203b-467c-b704-d4bd488f6c98"
+					(reference "R14")
+					(unit 1)
+				)
